Commit message: use_isaac_sim 모드 추가 (Isaac Sim 통합)
기존 use_fake_hardware / 실로봇 모드에 use_isaac_sim 분기 추가.
joint_state_topic_hardware_interface/JointStateTopicSystem plugin 으로
Isaac Sim 의 /joint_command, /joint_states 와 통신.

rbpodo_description/robots/rb_6dof.ros2_control.xacro:
- macro params 에 use_isaac_sim:=^|false 추가
- hardware plugin 3-way 분기:
  * use_isaac_sim=true → JointStateTopicSystem
    (joint_commands_topic=/joint_command, joint_states_topic=/joint_states,
     sum_wrapped_joint_states=true)
  * use_fake_hardware=true → mock_components/GenericSystem (기존)
  * 둘 다 false → rbpodo_hardware/RBPodoHardwareInterface (기존, 실로봇)
- configure_joint macro 에 isaac param 으로 분기:
  * isaac=true 일 때 command_interface=position 만, state_interface=position
    (initial_value=0.0) + velocity (effort 없음 — JointStateTopicSystem 호환)
  * isaac=false 일 때 기존 그대로 (effort/velocity/position command+state)

rbpodo_description/robots/rb10_1300e_u.urdf.xacro:
- use_isaac_sim arg 추가, rb_6dof_ros2_control 에 전달

rbpodo_moveit_config/launch/moveit.launch.py:
- use_isaac_sim LaunchConfiguration + DeclareLaunchArgument
- mappings dict 에 use_isaac_sim 전달
- ros2_control_node 에 remap joint_states → controller_manager/joint_states
  (Isaac Sim publisher 와 충돌 회피)

사용:
ros2 launch rbpodo_moveit_config moveit.launch.py \
    model_id:=rb10_1300e_u use_isaac_sim:=true use_fake_hardware:=false

Stage 5 시뮬 검증 통과 (minjea@minjea, 2026-05-13).

File: rbpodo_description/robots/rb10_1300e_u.urdf.xacro (robot description, xacro)
@@ -7,4 +7,5 @@
   <xacro:arg name="cb_simulation" default="true"/>
   <xacro:arg name="use_fake_hardware" default="true"/>
+  <xacro:arg name="use_isaac_sim" default="false"/>
   <xacro:arg name="fake_sensor_commands" default="false"/>
   <!-- torque_constant = actual_torque_constant * gear_ratio -->
@@ -16,4 +17,4 @@
   <xacro:property name="wrist3_tc" value="${1}" />
   <xacro:rb_6dof model_id="rb10_1300e_u" prefix="$(arg prefix)" tcp_name="tcp" tcp_xyz="0 -0.1153 0" tcp_rpy="0 0 0" />
-  <xacro:rb_6dof_ros2_control prefix="$(arg prefix)" robot_ip="$(arg robot_ip)" cb_simulation="$(arg cb_simulation)" use_fake_hardware="$(arg use_fake_hardware)" fake_sensor_commands="$(arg fake_sensor_commands)" torque_constants="${[base_tc, shoulder_tc, elbow_tc, wrist1_tc, wrist2_tc, wrist3_tc]}" />
+  <xacro:rb_6dof_ros2_control prefix="$(arg prefix)" robot_ip="$(arg robot_ip)" cb_simulation="$(arg cb_simulation)" use_fake_hardware="$(arg use_fake_hardware)" use_isaac_sim="$(arg use_isaac_sim)" fake_sensor_commands="$(arg fake_sensor_commands)" torque_constants="${[base_tc, shoulder_tc, elbow_tc, wrist1_tc, wrist2_tc, wrist3_tc]}" />
 </robot>

File: rbpodo_description/robots/rb_6dof.ros2_control.xacro (robot description, xacro)
@@ -1,35 +1,55 @@
 <?xml version='1.0' encoding='utf-8'?>
 <robot xmlns:xacro="http://www.ros.org/wiki/xacro">
-  <xacro:macro name="rb_6dof_ros2_control" params="prefix robot_ip cb_simulation:=^|false use_fake_hardware:=^|false fake_sensor_commands:=^|false torque_constants:=${[1, 1, 1, 1, 1, 1]}">
+  <xacro:macro name="rb_6dof_ros2_control" params="prefix robot_ip cb_simulation:=^|false use_fake_hardware:=^|false use_isaac_sim:=^|false fake_sensor_commands:=^|false torque_constants:=${[1, 1, 1, 1, 1, 1]}">
     <ros2_control name="RBPodoHardwareInterface" type="system">
       <hardware>
-        <xacro:if value="${use_fake_hardware}">
-          <plugin>mock_components/GenericSystem</plugin>
-          <param name="mock_sensor_commands">${fake_sensor_commands}</param>
-          <param name="state_following_offset">0.0</param>
+        <xacro:if value="${use_isaac_sim}">
+          <plugin>joint_state_topic_hardware_interface/JointStateTopicSystem</plugin>
+          <param name="joint_commands_topic">/joint_command</param>
+          <param name="joint_states_topic">/joint_states</param>
+          <param name="sum_wrapped_joint_states">true</param>
         </xacro:if>
-        <xacro:unless value="${use_fake_hardware}">
-          <plugin>rbpodo_hardware/RBPodoHardwareInterface</plugin>
-          <param name="cb_simulation">${cb_simulation}</param>
-          <param name="robot_ip">${robot_ip}</param>
+        <xacro:unless value="${use_isaac_sim}">
+          <xacro:if value="${use_fake_hardware}">
+            <plugin>mock_components/GenericSystem</plugin>
+            <param name="mock_sensor_commands">${fake_sensor_commands}</param>
+            <param name="state_following_offset">0.0</param>
+          </xacro:if>
+          <xacro:unless value="${use_fake_hardware}">
+            <plugin>rbpodo_hardware/RBPodoHardwareInterface</plugin>
+            <param name="cb_simulation">${cb_simulation}</param>
+            <param name="robot_ip">${robot_ip}</param>
+          </xacro:unless>
         </xacro:unless>
       </hardware>
-      <xacro:macro name="configure_joint" params="joint_name torque_constant:=1">
+      <xacro:macro name="configure_joint" params="joint_name torque_constant:=1 isaac:=false">
         <joint name="${joint_name}">
           <param name="initial_position">0.0</param>
           <param name="torque_constant">${torque_constant}</param>
-          <command_interface name="effort"/>
-          <command_interface name="velocity"/>
-          <command_interface name="position"/>
-          <state_interface name="position"/>
-          <state_interface name="effort"/>
+          <xacro:if value="${isaac}">
+            <!-- Isaac Sim: JointStateTopicSystem 은 position command 만 처리.
+                 state_interface 도 공식 형식 (position+initial_value, velocity) 만; effort 없음. -->
+            <command_interface name="position"/>
+            <state_interface name="position">
+              <param name="initial_value">0.0</param>
+            </state_interface>
+            <state_interface name="velocity"/>
+          </xacro:if>
+          <xacro:unless value="${isaac}">
+            <command_interface name="effort"/>
+            <command_interface name="velocity"/>
+            <command_interface name="position"/>
+            <state_interface name="position"/>
+            <state_interface name="velocity"/>
+            <state_interface name="effort"/>
+          </xacro:unless>
         </joint>
       </xacro:macro>
-      <xacro:configure_joint joint_name="${prefix}base" torque_constant="${torque_constants[0]}" />
-      <xacro:configure_joint joint_name="${prefix}shoulder" torque_constant="${torque_constants[1]}" />
-      <xacro:configure_joint joint_name="${prefix}elbow" torque_constant="${torque_constants[2]}" />
-      <xacro:configure_joint joint_name="${prefix}wrist1" torque_constant="${torque_constants[3]}" />
-      <xacro:configure_joint joint_name="${prefix}wrist2" torque_constant="${torque_constants[4]}" />
-      <xacro:configure_joint joint_name="${prefix}wrist3" torque_constant="${torque_constants[5]}" />
+      <xacro:configure_joint joint_name="${prefix}base"     torque_constant="${torque_constants[0]}" isaac="${use_isaac_sim}" />
+      <xacro:configure_joint joint_name="${prefix}shoulder" torque_constant="${torque_constants[1]}" isaac="${use_isaac_sim}" />
+      <xacro:configure_joint joint_name="${prefix}elbow"    torque_constant="${torque_constants[2]}" isaac="${use_isaac_sim}" />
+      <xacro:configure_joint joint_name="${prefix}wrist1"   torque_constant="${torque_constants[3]}" isaac="${use_isaac_sim}" />
+      <xacro:configure_joint joint_name="${prefix}wrist2"   torque_constant="${torque_constants[4]}" isaac="${use_isaac_sim}" />
+      <xacro:configure_joint joint_name="${prefix}wrist3"   torque_constant="${torque_constants[5]}" isaac="${use_isaac_sim}" />
     </ros2_control>
   </xacro:macro>
